File: STM32WB5mm_testBoard.kicad_pcb (KiCad board)
At the start: 2 copper layers, 31.5 x 99.1 mm, 24 parts, among them J1 FFMD-10-01, J2 ZW-40-XX-X-S-XXX-XXX, J3 ZW-40-XX-X-S-XXX-XXX, J4 MTMM-102-05-G-S-175, P1 0475890001, U1 STM32WB5MMG, U2 LD3985M33R_SOT23, U3 USBLC6-2P6

Commit message: 6
Parts:
- added J5: M20-9991246, M20-9991246:HARWIN_M20-9991246, F.Cu at (36.4, 113.4)
- added J6: M20-9991246, M20-9991246:HARWIN_M20-9991246, F.Cu at (36.4, 117.5)
- added J7: ZW-20-09-L-S-250-320, ZW-20-09-L-S-250-320:SAMTEC_ZW-20-09-L-S-250-320, F.Cu at (22.6, 105.2)
- added J8: ZW-20-09-L-S-250-320, ZW-20-09-L-S-250-320:SAMTEC_ZW-20-09-L-S-250-320, F.Cu at (22.6, 109.3)

Commit message: 7
Parts:
- removed J2, J3: ZW-40-XX-X-S-XXX-XXX, ZW-40-XX-X-S-XXX-XXX:SAMTEC_ZW-40-XX-X-S-XXX-XXX
- moved J8 125.5 mm to (120.9, 31.4), turned to -90 degrees
- moved P1 112.2 mm to (109.7, 148.4), turned to 0 degrees
- moved J7 104.6 mm to (97.1, 31.8), turned to -90 degrees
- moved J6 85.6 mm to (120.5, 133.7), turned to 90 degrees
- moved J5 64.6 mm to (97.5, 134.5), turned to -90 degrees
- moved J1 57.1 mm to (97.3, 99.2), turned to 90 degrees
- moved S2 8.38 mm to (109.9, 124.6)
